File: pcb layout/pcb layout.kicad_sch (KiCad schematic)
At the start: 7 parts, among them U1 ESP32-DevKitC, U2 DHT11

Commit message: feat: update pcb
Parts:
- Brd1: footprint Display:Adafruit_SSD1306 -> SSD1306:128x64OLED
Changed lines of the file:
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@@
 			)
 		)
-		(property "Footprint" "Display:Adafruit_SSD1306"
+		(property "Footprint" "SSD1306:128x64OLED"
 			(at 184.15 48.26 0)
 			(effects
